File: adc_blk.brd (EAGLE design)
At the start: 160 x 100 mm, 28 parts

Commit message: updates after cleaning up library references
Parts:
- removed ADC_BUFF1:U2: ADA4932-1YCPZ-R7, AD7960:CP_16_2
- added ADC_BUFF1:U3: AD7960BCPZ-RL7, open_covg:CP_32_7
- ADC_BUFF1:U1: value AD7960BCPZ-RL7 -> ADA4932-1YCPZ-R7; device AD7960:CP_32_7 -> open_covg:CP_16_2
- moved ADC_BUFF1:U1 57.7 mm to (-11.4, -162.6)
Connections:
- net ADC_BUFF1:+5V: now also ADC_BUFF1:U3.1, ADC_BUFF1:U3.19, ADC_BUFF1:U3.20; no longer ADC_BUFF1:U1.1, ADC_BUFF1:U1.19, ADC_BUFF1:U1.20
- net ADC_BUFF1:1.8V: now also ADC_BUFF1:U3.12, ADC_BUFF1:U3.2, ADC_BUFF1:U3.25; no longer ADC_BUFF1:U1.12, ADC_BUFF1:U1.2, ADC_BUFF1:U1.25
- net ADC_BUFF1:AMP_PWR+: now also ADC_BUFF1:U1.12, ADC_BUFF1:U1.5, ADC_BUFF1:U1.6, ADC_BUFF1:U1.7, ADC_BUFF1:U1.8; no longer ADC_BUFF1:U2.12, ADC_BUFF1:U2.5, ADC_BUFF1:U2.6, ADC_BUFF1:U2.7, ADC_BUFF1:U2.8
- net ADC_BUFF1:AMP_PWR-: now also ADC_BUFF1:U1.13, ADC_BUFF1:U1.14, ADC_BUFF1:U1.15, ADC_BUFF1:U1.16; no longer ADC_BUFF1:U2.13, ADC_BUFF1:U2.14, ADC_BUFF1:U2.15, ADC_BUFF1:U2.16
- net ADC_BUFF1:CLK+: now also ADC_BUFF1:U3.17; no longer ADC_BUFF1:U1.17
- net ADC_BUFF1:CLK-: now also ADC_BUFF1:U3.16; no longer ADC_BUFF1:U1.16
- net ADC_BUFF1:CNV+: now also ADC_BUFF1:U3.9; no longer ADC_BUFF1:U1.9
- net ADC_BUFF1:CNV-: now also ADC_BUFF1:U3.8; no longer ADC_BUFF1:U1.8
- net ADC_BUFF1:D+: now also ADC_BUFF1:U3.11; no longer ADC_BUFF1:U1.11
- net ADC_BUFF1:D-: now also ADC_BUFF1:U3.10; no longer ADC_BUFF1:U1.10
- net ADC_BUFF1:DCO+: now also ADC_BUFF1:U3.15; no longer ADC_BUFF1:U1.15
- net ADC_BUFF1:DCO-: now also ADC_BUFF1:U3.14; no longer ADC_BUFF1:U1.14
- net ADC_BUFF1:EN0: now also ADC_BUFF1:U3.4; no longer ADC_BUFF1:U1.4
- net ADC_BUFF1:EN1: now also ADC_BUFF1:U3.5; no longer ADC_BUFF1:U1.5
- net ADC_BUFF1:EN2: now also ADC_BUFF1:U3.6; no longer ADC_BUFF1:U1.6
- net ADC_BUFF1:EN3: now also ADC_BUFF1:U3.7; no longer ADC_BUFF1:U1.7
- net ADC_BUFF1:GND: now also ADC_BUFF1:U1.17, ADC_BUFF1:U3.13, ADC_BUFF1:U3.24, ADC_BUFF1:U3.26, ADC_BUFF1:U3.27, ADC_BUFF1:U3.28, ADC_BUFF1:U3.3, ADC_BUFF1:U3.HTAB; no longer ADC_BUFF1:U1.13, ADC_BUFF1:U1.24, ADC_BUFF1:U1.26, ADC_BUFF1:U1.27, ADC_BUFF1:U1.28, ADC_BUFF1:U1.3, ADC_BUFF1:U1.HTAB, ADC_BUFF1:U2.17
- net ADC_BUFF1:IN+: now also ADC_BUFF1:U3.23; no longer ADC_BUFF1:U1.23
- net ADC_BUFF1:IN-: now also ADC_BUFF1:U3.22; no longer ADC_BUFF1:U1.22
- net ADC_BUFF1:N$11: now also ADC_BUFF1:U1.2; no longer ADC_BUFF1:U2.2
- net ADC_BUFF1:N$12: now also ADC_BUFF1:U1.1; no longer ADC_BUFF1:U2.1
- net ADC_BUFF1:N$13: now also ADC_BUFF1:U1.3; no longer ADC_BUFF1:U2.3
- net ADC_BUFF1:N$14: now also ADC_BUFF1:U1.4; no longer ADC_BUFF1:U2.4
- net ADC_BUFF1:N$4: now also ADC_BUFF1:U3.18; no longer ADC_BUFF1:U1.18
- net ADC_BUFF1:N$5: now also ADC_BUFF1:U1.10; no longer ADC_BUFF1:U2.10
- net ADC_BUFF1:N$6: now also ADC_BUFF1:U1.11; no longer ADC_BUFF1:U2.11
- net ADC_BUFF1:REF: now also ADC_BUFF1:U3.29, ADC_BUFF1:U3.30, ADC_BUFF1:U3.31, ADC_BUFF1:U3.32; no longer ADC_BUFF1:U1.29, ADC_BUFF1:U1.30, ADC_BUFF1:U1.31, ADC_BUFF1:U1.32
- net ADC_BUFF1:VCM: now also ADC_BUFF1:U1.9, ADC_BUFF1:U3.21; no longer ADC_BUFF1:U1.21, ADC_BUFF1:U2.9
