File: adc2.sch (KiCad schematic (older format))
At the start: 31 parts, among them U21 ADA4932-1YCPZ-R7, U22 AD7960BCPZ-RL7, X3 BU-SMA-G, X4 BU-SMA-G

Commit message: cleanup from Eagle import
Parts:
- C55, C56, C57, C58, C59, C60, C61, C62, C63, C64, C65, C66, C67, C68: footprint adc_dac_v1:C0603 -> Capacitor_SMD:C_0603_1608Metric
- R53, R54, R55, R56, R57, R58, R59, R60, R61, R62, R63, R64: footprint adc_dac_v1:R0603 -> Resistor_SMD:R_0603_1608Metric
