File: adc3.sch (KiCad schematic (older format))
At the start: 31 parts, among them U25 ADA4932-1YCPZ-R7, U26 AD7960BCPZ-RL7, X5 BU-SMA-G, X6 BU-SMA-G

Commit message: cleanup from Eagle import
Parts:
- C69, C70, C71, C72, C73, C74, C75, C76, C77, C78, C79, C80, C81, C82: footprint adc_dac_v1:C0603 -> Capacitor_SMD:C_0603_1608Metric
- R78, R79, R80, R81, R82, R83, R84, R85, R86, R87, R88, R89: footprint adc_dac_v1:R0603 -> Resistor_SMD:R_0603_1608Metric
