File: adc4.sch (KiCad schematic (older format))
At the start: 34 parts, among them U27 ADA4932-1YCPZ-R7, U28 AD7960BCPZ-RL7, U36 AD8244BRMZ, X7 BU-SMA-G, X8 BU-SMA-G

Commit message: cleanup from Eagle import
Parts:
- C121, C122, C83, C84, C85, C86, C87, C88, C89, C90, C91, C92, C93, C94, C95, C96: footprint adc_dac_v1:C0603 -> Capacitor_SMD:C_0603_1608Metric
- R100, R101, R90, R91, R92, R93, R94, R95, R96, R97, R98, R99: footprint adc_dac_v1:R0603 -> Resistor_SMD:R_0603_1608Metric
