File: dac1.sch (KiCad schematic (older format))
At the start: 25 parts, among them IC1 OPA1662, IC3 ADA4610-2, J3 2-406541-3, U2 AD5453

Commit message: cleanup from Eagle import
Parts:
- C10, C23, C24, C3, C6, C7, C8, C9: footprint adc_dac_v1:C0603 -> Capacitor_SMD:C_0603_1608Metric; symbol adc_dac_v1-eagle-import:C-USC0603 -> Device:C
- R1, R14, R148, R149, R150, R2, R21, R22, R3, R4, R5, R6, R7: footprint adc_dac_v1:R0603 -> Resistor_SMD:R_0603_1608Metric; symbol adc_dac_v1-eagle-import:R-US_R0603 -> Device:R_US
Connections:
- net labels added: +3V3
- net labels removed: 3V3, N$10, N$2, N$3, N$4, N$5, N$7, N$8
- wire segments 84 -> 91
Other:
- moved on the sheet: IC1B, IC3A, IC3B, IC3C
