File: dac2.sch (KiCad schematic (older format))
At the start: 24 parts, among them IC2 ADA4610-2, IC4 OPA1662, U29 AD5453YRMZ-REEL7

Commit message: cleanup from Eagle import
Parts:
- C100, C101, C102, C103, C104, C97, C98, C99: footprint adc_dac_v1:C0603 -> Capacitor_SMD:C_0603_1608Metric
- R102, R103, R104, R105, R106, R107, R108, R109, R110, R111, R139, R140, R141: footprint adc_dac_v1:R0603 -> Resistor_SMD:R_0603_1608Metric
