File: dac3.sch (KiCad schematic (older format))
At the start: 24 parts, among them IC5 ADA4610-2, IC6 OPA1662, U30 AD5453

Commit message: cleanup from Eagle import
Parts:
- C105, C106, C107, C108, C109, C110, C111, C112: footprint adc_dac_v1:C0603 -> Capacitor_SMD:C_0603_1608Metric
- R112, R113, R114, R115, R116, R117, R118, R119, R120, R121, R142, R143, R144: footprint adc_dac_v1:R0603 -> Resistor_SMD:R_0603_1608Metric
