File: dac4.sch (KiCad schematic (older format))
At the start: 24 parts, among them IC7 ADA4610-2, IC8 OPA1662, U32 AD5453

Commit message: cleanup from Eagle import
Parts:
- C113, C114, C115, C116, C117, C118, C119, C120: footprint adc_dac_v1:C0603 -> Capacitor_SMD:C_0603_1608Metric
- R122, R123, R124, R125, R126, R127, R128, R129, R130, R131, R145, R146, R147: footprint adc_dac_v1:R0603 -> Resistor_SMD:R_0603_1608Metric
