File: howland_ipump.sch (KiCad schematic (older format))
At the start: 13 parts, among them Q1 BC856, U11 OPA991S

Commit message: after using kifield to update Manf#
Parts:
- C34: Manufacturer_Name (none) -> Yageo; voltage 25V -> 25
- C35: Manufacturer_Name (none) -> Yageo; Tolerance (none) -> 20%; voltage 25V -> 25
- Q1: Manf# (none) -> BC856B-7-F
- R27: Power (none) -> 0.1W; Tolerance 0.1 -> 1%
- R53, R54: Power (none) -> 0.1W; Tolerance 0.1 -> (none)
- U11: Manf# (none) -> OPA991SIDBVR
