File: howland_ipump.sch (KiCad schematic (older format))
At the start: 13 parts, among them Q1 BC856, U12 OPA991S

Commit message: rolled back to commit b6c4f66 because of rescue libraries
Parts:
- C11, C12, C13: symbol covg_daq_v2-rescue:C-Device -> Device:C
- Q1: symbol covg_daq_v2-rescue:BC856-Transistor_BJT -> Transistor_BJT:BC856
- R27, R28, R29, R30, R31, R32, R33, R34: symbol covg_daq_v2-rescue:R_US-Device -> Device:R_US
- U12: symbol covg_daq_v2-rescue:OPA991S-covg-kicad -> covg-kicad:OPA991S
Changed lines of the file:
@@
 $Descr A4 11693 8268
 encoding utf-8
-Sheet 3 26
+Sheet 22 26
 Title ""
 Date ""
@@
 $EndDescr
 $Comp
-L covg_daq_v2-rescue:-15V-power #PWR?
+L power:-15V #PWR?
 U 1 1 60D781E3
 P 5100 4050
@@
 $EndComp
 $Comp
-L covg_daq_v2-rescue:+15V-power #PWR?
+L power:+15V #PWR?
 U 1 1 60D781E9
 P 5100 3400
@@
 $EndComp
 $Comp
-L covg_daq_v2-rescue:C-Device C?
+L Device:C C?
 U 1 1 60D781F4
 P 5850 4500
@@
 $EndComp
 $Comp
-L covg_daq_v2-rescue:GND-power #PWR?
+L power:GND #PWR?
 U 1 1 60D78215
 P 3650 3900
@@
 $EndComp
 $Comp
-L covg_daq_v2-rescue:OPA991S-covg-kicad U?
+L covg-kicad:OPA991S U?
 U 1 1 60D7821F
 P 5200 3700
@@
 $EndComp
 $Comp
-L covg_daq_v2-rescue:R_US-Device R?
+L Device:R_US R?
 U 1 1 60D78240
 P 5850 4950
@@
 $EndComp
 $Comp
-L covg_daq_v2-rescue:C-Device C?
+L Device:C C?
 U 1 1 60D7824A
 P 6750 3650
@@
 $EndComp
 $Comp
-L covg_daq_v2-rescue:GND-power #PWR?
+L power:GND #PWR?
 U 1 1 60D78250
 P 6750 3900
@@
 $EndComp
 $Comp
-L covg_daq_v2-rescue:+15V-power #PWR?
+L power:+15V #PWR?
 U 1 1 60D78256
 P 7150 3400
@@
 $EndComp
 $Comp
-L covg_daq_v2-rescue:GND-power #PWR?
+L power:GND #PWR?
 U 1 1 60D7825C
 P 7150 3900
@@
 $EndComp
 $Comp
-L covg_daq_v2-rescue:C-Device C?
+L Device:C C?
 U 1 1 60D78264
 P 7150 3650
@@
 $EndComp
 $Comp
-L covg_daq_v2-rescue:-15V-power #PWR?
+L power:-15V #PWR?
 U 1 1 60D7826A
 P 6750 3400
@@
 $EndComp
 $Comp
-L covg_daq_v2-rescue:R_US-Device R?
+L Device:R_US R?
 U 1 1 60D83006
 P 4300 3800
@@
 $EndComp
 $Comp
-L covg_daq_v2-rescue:R_US-Device R?
+L Device:R_US R?
 U 1 1 60D8879F
 P 4300 3600
@@
 $EndComp
 $Comp
-L covg_daq_v2-rescue:R_US-Device R?
+L Device:R_US R?
 U 1 1 60B385AE
 P 3800 3800
@@
 $EndComp
 $Comp
-L covg_daq_v2-rescue:R_US-Device R?
+L Device:R_US R?
 U 1 1 60B38EA4
 P 3750 3600
@@
 $EndComp
 $Comp
-L covg_daq_v2-rescue:R_US-Device R?
+L Device:R_US R?
 U 1 1 60B3940D
 P 5400 3000
@@
 $EndComp
 $Comp
-L covg_daq_v2-rescue:BC856-Transistor_BJT Q1
+L Transistor_BJT:BC856 Q1
 U 1 1 60BEDC00
 P 7750 4050
@@
 $EndComp
 $Comp
-L covg_daq_v2-rescue:R_US-Device R?
+L Device:R_US R?
 U 1 1 60BF0E09
 P 8200 4050
@@
 $EndComp
 $Comp
-L covg_daq_v2-rescue:+3V3-power #PWR064
+L power:+3V3 #PWR064
 U 1 1 60BF2F91
 P 7650 3250
@@
 $EndComp
 $Comp
-L covg_daq_v2-rescue:R_US-Device R?
+L Device:R_US R?
 U 1 1 60C16A39
 P 7950 3750

Commit message: DC-DC Regulator updated
Parts:
- C11, C12, C13: symbol Device:C -> covg_daq_v2-rescue:C-Device
- Q1: symbol Transistor_BJT:BC856 -> covg_daq_v2-rescue:BC856-Transistor_BJT
- R27, R28, R29, R30, R31, R32, R33, R34: symbol Device:R_US -> covg_daq_v2-rescue:R_US-Device
- U12: symbol covg-kicad:OPA991S -> covg_daq_v2-rescue:OPA991S-covg-kicad
Changed lines of the file:
@@
 $EndDescr
 $Comp
-L power:-15V #PWR?
+L covg_daq_v2-rescue:-15V-power #PWR?
 U 1 1 60D781E3
 P 5100 4050
@@
 $EndComp
 $Comp
-L power:+15V #PWR?
+L covg_daq_v2-rescue:+15V-power #PWR?
 U 1 1 60D781E9
 P 5100 3400
@@
 $EndComp
 $Comp
-L Device:C C?
+L covg_daq_v2-rescue:C-Device C?
 U 1 1 60D781F4
 P 5850 4500
@@
 $EndComp
 $Comp
-L power:GND #PWR?
+L covg_daq_v2-rescue:GND-power #PWR?
 U 1 1 60D78215
 P 3650 3900
@@
 $EndComp
 $Comp
-L covg-kicad:OPA991S U?
+L covg_daq_v2-rescue:OPA991S-covg-kicad U?
 U 1 1 60D7821F
 P 5200 3700
@@
 $EndComp
 $Comp
-L Device:R_US R?
+L covg_daq_v2-rescue:R_US-Device R?
 U 1 1 60D78240
 P 5850 4950
@@
 $EndComp
 $Comp
-L Device:C C?
+L covg_daq_v2-rescue:C-Device C?
 U 1 1 60D7824A
 P 6750 3650
@@
 $EndComp
 $Comp
-L power:GND #PWR?
+L covg_daq_v2-rescue:GND-power #PWR?
 U 1 1 60D78250
 P 6750 3900
@@
 $EndComp
 $Comp
-L power:+15V #PWR?
+L covg_daq_v2-rescue:+15V-power #PWR?
 U 1 1 60D78256
 P 7150 3400
@@
 $EndComp
 $Comp
-L power:GND #PWR?
+L covg_daq_v2-rescue:GND-power #PWR?
 U 1 1 60D7825C
 P 7150 3900
@@
 $EndComp
 $Comp
-L Device:C C?
+L covg_daq_v2-rescue:C-Device C?
 U 1 1 60D78264
 P 7150 3650
@@
 $EndComp
 $Comp
-L power:-15V #PWR?
+L covg_daq_v2-rescue:-15V-power #PWR?
 U 1 1 60D7826A
 P 6750 3400
@@
 $EndComp
 $Comp
-L Device:R_US R?
+L covg_daq_v2-rescue:R_US-Device R?
 U 1 1 60D83006
 P 4300 3800
@@
 $EndComp
 $Comp
-L Device:R_US R?
+L covg_daq_v2-rescue:R_US-Device R?
 U 1 1 60D8879F
 P 4300 3600
@@
 $EndComp
 $Comp
-L Device:R_US R?
+L covg_daq_v2-rescue:R_US-Device R?
 U 1 1 60B385AE
 P 3800 3800
@@
 $EndComp
 $Comp
-L Device:R_US R?
+L covg_daq_v2-rescue:R_US-Device R?
 U 1 1 60B38EA4
 P 3750 3600
@@
 $EndComp
 $Comp
-L Device:R_US R?
+L covg_daq_v2-rescue:R_US-Device R?
 U 1 1 60B3940D
 P 5400 3000
@@
 $EndComp
 $Comp
-L Transistor_BJT:BC856 Q1
+L covg_daq_v2-rescue:BC856-Transistor_BJT Q1
 U 1 1 60BEDC00
 P 7750 4050
@@
 $EndComp
 $Comp
-L Device:R_US R?
+L covg_daq_v2-rescue:R_US-Device R?
 U 1 1 60BF0E09
 P 8200 4050
@@
 $EndComp
 $Comp
-L power:+3V3 #PWR064
+L covg_daq_v2-rescue:+3V3-power #PWR064
 U 1 1 60BF2F91
 P 7650 3250
@@
 $EndComp
 $Comp
-L Device:R_US R?
+L covg_daq_v2-rescue:R_US-Device R?
 U 1 1 60C16A39
 P 7950 3750
