File: dual_bipolar_amp.sch (KiCad schematic (older format))
At the start: 9 parts, among them U4 OPA2156xD

Commit message: DC-DC Regulator updated
Parts:
- C174, C175: symbol Device:C -> covg_daq_v2-rescue:C-Device
- R84, R85, R86, R87, R88, R89: symbol Device:R_US -> covg_daq_v2-rescue:R_US-Device
- U4: symbol Amplifier_Operational:OPA2156xD -> covg_daq_v2-rescue:OPA2156xD-Amplifier_Operational
Changed lines of the file:
@@
 $EndDescr
 $Comp
-L Amplifier_Operational:OPA2156xD U?
+L covg_daq_v2-rescue:OPA2156xD-Amplifier_Operational U?
 U 1 1 60F31C8B
 P 5600 3250
@@
 AR Path="/6095BD4C/60EB6FD5/60F31C8B" Ref="U2"  Part="1"
 AR Path="/61B02572/60EB6FD5/60F31C8B" Ref="U9"  Part="1"
+AR Path="/60F31C8B" Ref="U9"  Part="1"
 F 0 "U9" H 5600 3617 50  0000 C CNN
 F 1 "OPA2156xD" H 5600 3526 50  0000 C CNN
@@
 $EndComp
 $Comp
-L Device:R_US R?
+L covg_daq_v2-rescue:R_US-Device R?
 U 1 1 60F31C94
 P 4800 3350
@@
 $EndComp
 $Comp
-L Amplifier_Operational:OPA2156xD U?
+L covg_daq_v2-rescue:OPA2156xD-Amplifier_Operational U?
 U 3 1 60F31C9B
 P 4750 2300
@@
 AR Path="/6095BD4C/60EB6FD5/60F31C9B" Ref="U2"  Part="3"
 AR Path="/61B02572/60EB6FD5/60F31C9B" Ref="U9"  Part="3"
+AR Path="/60F31C9B" Ref="U9"  Part="3"
 F 0 "U9" H 4808 2346 50  0000 L CNN
 F 1 "OPA2156xD" H 4808 2255 50  0000 L CNN
@@
 $EndComp
 $Comp
-L Device:R_US R?
+L covg_daq_v2-rescue:R_US-Device R?
 U 1 1 60F31CA4
 P 4900 3650
@@
 $EndComp
 $Comp
-L power:GND #GND?
+L covg_daq_v2-rescue:GND-power #GND?
 U 1 1 60F31CAA
 P 4700 3800
@@
 $EndComp
 $Comp
-L Device:R_US R?
+L covg_daq_v2-rescue:R_US-Device R?
 U 1 1 60F31CB1
 P 5550 3650
@@
 $EndComp
 $Comp
-L Amplifier_Operational:OPA2156xD U?
+L covg_daq_v2-rescue:OPA2156xD-Amplifier_Operational U?
 U 2 1 60F31CB8
 P 5600 4200
@@
 AR Path="/6095BD4C/60EB6FD5/60F31CB8" Ref="U2"  Part="2"
 AR Path="/61B02572/60EB6FD5/60F31CB8" Ref="U9"  Part="2"
+AR Path="/60F31CB8" Ref="U9"  Part="2"
 F 0 "U9" H 5600 4567 50  0000 C CNN
 F 1 "OPA2156xD" H 5600 4476 50  0000 C CNN
@@
 $EndComp
 $Comp
-L Device:R_US R?
+L covg_daq_v2-rescue:R_US-Device R?
 U 1 1 60F31CC1
 P 4800 4300
@@
 $EndComp
 $Comp
-L Device:R_US R?
+L covg_daq_v2-rescue:R_US-Device R?
 U 1 1 60F31CCA
 P 4900 4600
@@
 $EndComp
 $Comp
-L power:GND #GND?
+L covg_daq_v2-rescue:GND-power #GND?
 U 1 1 60F31CD0
 P 4700 4750
@@
 $EndComp
 $Comp
-L Device:R_US R?
+L covg_daq_v2-rescue:R_US-Device R?
 U 1 1 60F31CD7
 P 5550 4600
@@
 $EndComp
 $Comp
-L power:+15V #PWR?
+L covg_daq_v2-rescue:+15V-power #PWR?
 U 1 1 60F31CDD
 P 4750 1950
@@
 $EndComp
 $Comp
-L power:-15V #PWR?
+L covg_daq_v2-rescue:-15V-power #PWR?
 U 1 1 60F31CE3
 P 4750 2700
@@
 $EndComp
 $Comp
-L Device:C C?
+L covg_daq_v2-rescue:C-Device C?
 U 1 1 60F31CED
 P 5400 2250
@@
 $EndComp
 $Comp
-L Device:C C?
+L covg_daq_v2-rescue:C-Device C?
 U 1 1 60F31CF7
 P 5800 2250
@@
 $EndComp
 $Comp
-L power:-15V #PWR?
+L covg_daq_v2-rescue:-15V-power #PWR?
 U 1 1 60F31CFD
 P 5400 2500
@@
 $EndComp
 $Comp
-L power:GND #GND?
+L covg_daq_v2-rescue:GND-power #GND?
 U 1 1 60F31D03
 P 5400 2000
@@
 $EndComp
 $Comp
-L power:+15V #PWR?
+L covg_daq_v2-rescue:+15V-power #PWR?
 U 1 1 60F31D09
 P 5800 2000
@@
 $EndComp
 $Comp
-L power:GND #GND?
+L covg_daq_v2-rescue:GND-power #GND?
 U 1 1 60F31D0F
 P 5800 2550

Commit message: rolled back to commit b6c4f66 because of rescue libraries
Parts:
- C174, C175: symbol covg_daq_v2-rescue:C-Device -> Device:C
- R84, R85, R86, R87, R88, R89: symbol covg_daq_v2-rescue:R_US-Device -> Device:R_US
- U4: symbol covg_daq_v2-rescue:OPA2156xD-Amplifier_Operational -> Amplifier_Operational:OPA2156xD
Changed lines of the file:
@@
 $EndDescr
 $Comp
-L covg_daq_v2-rescue:OPA2156xD-Amplifier_Operational U?
+L Amplifier_Operational:OPA2156xD U?
 U 1 1 60F31C8B
 P 5600 3250
@@
 AR Path="/6095BD4C/60EB6FD5/60F31C8B" Ref="U2"  Part="1"
 AR Path="/61B02572/60EB6FD5/60F31C8B" Ref="U9"  Part="1"
-AR Path="/60F31C8B" Ref="U9"  Part="1"
 F 0 "U9" H 5600 3617 50  0000 C CNN
 F 1 "OPA2156xD" H 5600 3526 50  0000 C CNN
@@
 $EndComp
 $Comp
-L covg_daq_v2-rescue:R_US-Device R?
+L Device:R_US R?
 U 1 1 60F31C94
 P 4800 3350
@@
 $EndComp
 $Comp
-L covg_daq_v2-rescue:OPA2156xD-Amplifier_Operational U?
+L Amplifier_Operational:OPA2156xD U?
 U 3 1 60F31C9B
 P 4750 2300
@@
 AR Path="/6095BD4C/60EB6FD5/60F31C9B" Ref="U2"  Part="3"
 AR Path="/61B02572/60EB6FD5/60F31C9B" Ref="U9"  Part="3"
-AR Path="/60F31C9B" Ref="U9"  Part="3"
 F 0 "U9" H 4808 2346 50  0000 L CNN
 F 1 "OPA2156xD" H 4808 2255 50  0000 L CNN
@@
 $EndComp
 $Comp
-L covg_daq_v2-rescue:R_US-Device R?
+L Device:R_US R?
 U 1 1 60F31CA4
 P 4900 3650
@@
 $EndComp
 $Comp
-L covg_daq_v2-rescue:GND-power #GND?
+L power:GND #GND?
 U 1 1 60F31CAA
 P 4700 3800
@@
 $EndComp
 $Comp
-L covg_daq_v2-rescue:R_US-Device R?
+L Device:R_US R?
 U 1 1 60F31CB1
 P 5550 3650
@@
 $EndComp
 $Comp
-L covg_daq_v2-rescue:OPA2156xD-Amplifier_Operational U?
+L Amplifier_Operational:OPA2156xD U?
 U 2 1 60F31CB8
 P 5600 4200
@@
 AR Path="/6095BD4C/60EB6FD5/60F31CB8" Ref="U2"  Part="2"
 AR Path="/61B02572/60EB6FD5/60F31CB8" Ref="U9"  Part="2"
-AR Path="/60F31CB8" Ref="U9"  Part="2"
 F 0 "U9" H 5600 4567 50  0000 C CNN
 F 1 "OPA2156xD" H 5600 4476 50  0000 C CNN
@@
 $EndComp
 $Comp
-L covg_daq_v2-rescue:R_US-Device R?
+L Device:R_US R?
 U 1 1 60F31CC1
 P 4800 4300
@@
 $EndComp
 $Comp
-L covg_daq_v2-rescue:R_US-Device R?
+L Device:R_US R?
 U 1 1 60F31CCA
 P 4900 4600
@@
 $EndComp
 $Comp
-L covg_daq_v2-rescue:GND-power #GND?
+L power:GND #GND?
 U 1 1 60F31CD0
 P 4700 4750
@@
 $EndComp
 $Comp
-L covg_daq_v2-rescue:R_US-Device R?
+L Device:R_US R?
 U 1 1 60F31CD7
 P 5550 4600
@@
 $EndComp
 $Comp
-L covg_daq_v2-rescue:+15V-power #PWR?
+L power:+15V #PWR?
 U 1 1 60F31CDD
 P 4750 1950
@@
 $EndComp
 $Comp
-L covg_daq_v2-rescue:-15V-power #PWR?
+L power:-15V #PWR?
 U 1 1 60F31CE3
 P 4750 2700
@@
 $EndComp
 $Comp
-L covg_daq_v2-rescue:C-Device C?
+L Device:C C?
 U 1 1 60F31CED
 P 5400 2250
@@
 $EndComp
 $Comp
-L covg_daq_v2-rescue:C-Device C?
+L Device:C C?
 U 1 1 60F31CF7
 P 5800 2250
@@
 $EndComp
 $Comp
-L covg_daq_v2-rescue:-15V-power #PWR?
+L power:-15V #PWR?
 U 1 1 60F31CFD
 P 5400 2500
@@
 $EndComp
 $Comp
-L covg_daq_v2-rescue:GND-power #GND?
+L power:GND #GND?
 U 1 1 60F31D03
 P 5400 2000
@@
 $EndComp
 $Comp
-L covg_daq_v2-rescue:+15V-power #PWR?
+L power:+15V #PWR?
 U 1 1 60F31D09
 P 5800 2000
@@
 $EndComp
 $Comp
-L covg_daq_v2-rescue:GND-power #GND?
+L power:GND #GND?
 U 1 1 60F31D0F
 P 5800 2550
