File: power.sch (KiCad schematic (older format))
At the start: 57 parts, among them J12 Barrel_Jack_Switch, J13 Conn_02x05_Odd_Even, J14 Screw_Terminal_01x12, U13 LT3471, U14 LP38692MP-5.0, U15 LP38693MP-3.3, U16 LM2937xMP, U17 MAX6070BAUT21+T, U18 LP38693MP-1.8, U19 MC79M15_TO252, U20 LP38693MP-2.5

Commit message: move bom files to bom folder
Parts:
- C15, C21, C24, C28, C30, C33, C36, C37: Manf# CL10B105MO8NNWC -> CL10A105KA8NFNC; Tolerance 20% -> 10%; voltage 16V -> 25V
- C20: Manf# GMK107BJ105KA-T -> CL10A105KA8NFNC; voltage 35V -> 25V
Changed lines of the file:
@@
 F 2 "Capacitor_SMD:C_0603_1608Metric" H 2000 2550 50  0001 C CNN
 F 3 "" H 2000 2550 50  0001 C CNN
-F 4 "CL10B105MO8NNWC" H 2040 2675 50  0001 C CNN "Manf#"
-F 5 "20%" H 2040 2675 50  0001 C CNN "Tolerance"
-F 6 "16V" H 2040 2675 50  0001 C CNN "voltage"
+F 4 "CL10A105KA8NFNC" H 2040 2675 50  0001 C CNN "Manf#"
+F 5 "10%" H 2040 2675 50  0001 C CNN "Tolerance"
+F 6 "25V" H 2040 2675 50  0001 C CNN "voltage"
 	1    2000 2550
 	1    0    0    -1
@@
 F 2 "Capacitor_SMD:C_0603_1608Metric" H 3600 4100 50  0001 C CNN
 F 3 "" H 3600 4100 50  0001 C CNN
-F 4 "GMK107BJ105KA-T" H 3640 4225 50  0001 C CNN "Manf#"
+F 4 "CL10A105KA8NFNC" H 3640 4225 50  0001 C CNN "Manf#"
 F 5 "10%" H 3640 4225 50  0001 C CNN "Tolerance"
-F 6 "35V" H 3640 4225 50  0001 C CNN "voltage"
+F 6 "25V" H 3640 4225 50  0001 C CNN "voltage"
 	1    3600 4100
 	0    1    1    0
@@
 F 2 "Capacitor_SMD:C_0603_1608Metric" H 4900 2550 50  0001 C CNN
 F 3 "" H 4900 2550 50  0001 C CNN
-F 4 "CL10B105MO8NNWC" H 4940 2675 50  0001 C CNN "Manf#"
-F 5 "20%" H 4940 2675 50  0001 C CNN "Tolerance"
-F 6 "16V" H 4940 2675 50  0001 C CNN "voltage"
+F 4 "CL10A105KA8NFNC" H 4940 2675 50  0001 C CNN "Manf#"
+F 5 "10%" H 4940 2675 50  0001 C CNN "Tolerance"
+F 6 "25V" H 4940 2675 50  0001 C CNN "voltage"
 	1    4900 2550
 	1    0    0    -1
@@
 F 2 "Capacitor_SMD:C_0603_1608Metric" H 3850 2550 50  0001 C CNN
 F 3 "" H 3850 2550 50  0001 C CNN
-F 4 "CL10B105MO8NNWC" H 3890 2675 50  0001 C CNN "Manf#"
-F 5 "20%" H 3890 2675 50  0001 C CNN "Tolerance"
-F 6 "16V" H 3890 2675 50  0001 C CNN "voltage"
+F 4 "CL10A105KA8NFNC" H 3890 2675 50  0001 C CNN "Manf#"
+F 5 "10%" H 3890 2675 50  0001 C CNN "Tolerance"
+F 6 "25V" H 3890 2675 50  0001 C CNN "voltage"
 	1    3850 2550
 	1    0    0    -1
@@
 F 2 "Capacitor_SMD:C_0603_1608Metric" H 6700 2550 50  0001 C CNN
 F 3 "" H 6700 2550 50  0001 C CNN
-F 4 "CL10B105MO8NNWC" H 6740 2675 50  0001 C CNN "Manf#"
-F 5 "20%" H 6740 2675 50  0001 C CNN "Tolerance"
-F 6 "16V" H 6740 2675 50  0001 C CNN "voltage"
+F 4 "CL10A105KA8NFNC" H 6740 2675 50  0001 C CNN "Manf#"
+F 5 "10%" H 6740 2675 50  0001 C CNN "Tolerance"
+F 6 "25V" H 6740 2675 50  0001 C CNN "voltage"
 	1    6700 2550
 	1    0    0    -1
@@
 F 2 "Capacitor_SMD:C_0603_1608Metric" H 7200 2600 50  0001 C CNN
 F 3 "" H 7200 2600 50  0001 C CNN
-F 4 "CL10B105MO8NNWC" H 7240 2725 50  0001 C CNN "Manf#"
-F 5 "20%" H 7240 2725 50  0001 C CNN "Tolerance"
-F 6 "16V" H 7240 2725 50  0001 C CNN "voltage"
+F 4 "CL10A105KA8NFNC" H 7240 2725 50  0001 C CNN "Manf#"
+F 5 "10%" H 7240 2725 50  0001 C CNN "Tolerance"
+F 6 "25V" H 7240 2725 50  0001 C CNN "voltage"
 	1    7200 2600
 	1    0    0    -1
@@
 F 2 "Capacitor_SMD:C_0603_1608Metric" H 8850 2550 50  0001 C CNN
 F 3 "" H 8850 2550 50  0001 C CNN
-F 4 "CL10B105MO8NNWC" H 8890 2675 50  0001 C CNN "Manf#"
-F 5 "20%" H 8890 2675 50  0001 C CNN "Tolerance"
-F 6 "16V" H 8890 2675 50  0001 C CNN "voltage"
+F 4 "CL10A105KA8NFNC" H 8890 2675 50  0001 C CNN "Manf#"
+F 5 "10%" H 8890 2675 50  0001 C CNN "Tolerance"
+F 6 "25V" H 8890 2675 50  0001 C CNN "voltage"
 	1    8850 2550
 	1    0    0    -1
@@
 F 2 "Capacitor_SMD:C_0603_1608Metric" H 10000 2550 50  0001 C CNN
 F 3 "" H 10000 2550 50  0001 C CNN
-F 4 "CL10B105MO8NNWC" H 10040 2675 50  0001 C CNN "Manf#"
-F 5 "20%" H 10040 2675 50  0001 C CNN "Tolerance"
-F 6 "16V" H 10040 2675 50  0001 C CNN "voltage"
+F 4 "CL10A105KA8NFNC" H 10040 2675 50  0001 C CNN "Manf#"
+F 5 "10%" H 10040 2675 50  0001 C CNN "Tolerance"
+F 6 "25V" H 10040 2675 50  0001 C CNN "voltage"
 	1    10000 2550
 	1    0    0    -1
@@
 F 2 "Capacitor_SMD:C_0603_1608Metric" H 11500 2550 50  0001 C CNN
 F 3 "" H 11500 2550 50  0001 C CNN
-F 4 "CL10B105MO8NNWC" H 11540 2675 50  0001 C CNN "Manf#"
-F 5 "20%" H 11540 2675 50  0001 C CNN "Tolerance"
-F 6 "16V" H 11540 2675 50  0001 C CNN "voltage"
+F 4 "CL10A105KA8NFNC" H 11540 2675 50  0001 C CNN "Manf#"
+F 5 "10%" H 11540 2675 50  0001 C CNN "Tolerance"
+F 6 "25V" H 11540 2675 50  0001 C CNN "voltage"
 	1    11500 2550
 	1    0    0    -1
