File: junk/adc_backup.sch (KiCad schematic (older format))
At the start: 19 parts, among them J15 Conn_01x04_Male, U22 AD7960BCPZ-RL7, U23 OPA325

Commit message: changed 0.1uF cap to Samsung
Parts:
- C13, C14, C15, C18, C19, C23, C27: Manf# CL10B104KA8NFNC -> CC0603MRX7R8BB104; Manufacturer_Name Samsung -> Yageo; Tolerance 10% -> 20%
- C24: value 100p -> 2p; Manf# CC0603JRNPO0BN101 -> CC0603CRNPO9BN2R0; Tolerance 5% -> 0.25pF; voltage 100V -> 50V
Changed lines of the file:
@@
 AR Path="/60C1F416/B0DC2316" Ref="C112"  Part="1"
 F 0 "C24" H 7090 3725 59  0000 L BNN
-F 1 "100p" H 7090 3535 59  0000 L BNN
+F 1 "2p" H 7090 3535 59  0000 L BNN
 F 2 "Capacitor_SMD:C_0603_1608Metric" H 7050 3700 50  0001 C CNN
 F 3 "" H 7050 3700 50  0001 C CNN
-F 4 "CC0603JRNPO0BN101" H 7090 3825 50  0001 C CNN "Manf#"
-F 5 "5%" H 7090 3825 50  0001 C CNN "Tolerance"
-F 6 "100V" H 7090 3825 50  0001 C CNN "voltage"
+F 4 "CC0603CRNPO9BN2R0" H 7090 3825 50  0001 C CNN "Manf#"
+F 5 "0.25pF" H 7090 3825 50  0001 C CNN "Tolerance"
+F 6 "50V" H 7090 3825 50  0001 C CNN "voltage"
 	1    7050 3700
 	-1   0    0    -1
@@
 F 2 "Capacitor_SMD:C_0603_1608Metric" H 5350 2750 50  0001 C CNN
 F 3 "" H 5350 2750 50  0001 C CNN
-F 4 "CL10B104KA8NFNC" H 5390 2875 50  0001 C CNN "Manf#"
-F 5 "Samsung" H 5390 2875 50  0001 C CNN "Manufacturer_Name"
-F 6 "10%" H 5390 2875 50  0001 C CNN "Tolerance"
+F 4 "CC0603MRX7R8BB104" H 5390 2875 50  0001 C CNN "Manf#"
+F 5 "Yageo" H 5390 2875 50  0001 C CNN "Manufacturer_Name"
+F 6 "20%" H 5390 2875 50  0001 C CNN "Tolerance"
 F 7 "25" H 5390 2875 50  0001 C CNN "voltage"
 	1    5350 2750
@@
 F 2 "Capacitor_SMD:C_0603_1608Metric" H 5400 4300 50  0001 C CNN
 F 3 "" H 5400 4300 50  0001 C CNN
-F 4 "CL10B104KA8NFNC" H 5440 4425 50  0001 C CNN "Manf#"
-F 5 "Samsung" H 5440 4425 50  0001 C CNN "Manufacturer_Name"
-F 6 "10%" H 5440 4425 50  0001 C CNN "Tolerance"
+F 4 "CC0603MRX7R8BB104" H 5440 4425 50  0001 C CNN "Manf#"
+F 5 "Yageo" H 5440 4425 50  0001 C CNN "Manufacturer_Name"
+F 6 "20%" H 5440 4425 50  0001 C CNN "Tolerance"
 F 7 "25" H 5440 4425 50  0001 C CNN "voltage"
 	1    5400 4300
@@
 F 2 "Capacitor_SMD:C_0603_1608Metric" H 1450 3400 50  0001 C CNN
 F 3 "" H 1450 3400 50  0001 C CNN
-F 4 "CL10B104KA8NFNC" H 1490 3525 50  0001 C CNN "Manf#"
-F 5 "Samsung" H 1490 3525 50  0001 C CNN "Manufacturer_Name"
-F 6 "10%" H 1490 3525 50  0001 C CNN "Tolerance"
+F 4 "CC0603MRX7R8BB104" H 1490 3525 50  0001 C CNN "Manf#"
+F 5 "Yageo" H 1490 3525 50  0001 C CNN "Manufacturer_Name"
+F 6 "20%" H 1490 3525 50  0001 C CNN "Tolerance"
 F 7 "25" H 1490 3525 50  0001 C CNN "voltage"
 	1    1450 3400
@@
 F 2 "Capacitor_SMD:C_0603_1608Metric" H 1850 3400 50  0001 C CNN
 F 3 "" H 1850 3400 50  0001 C CNN
-F 4 "CL10B104KA8NFNC" H 1890 3525 50  0001 C CNN "Manf#"
-F 5 "Samsung" H 1890 3525 50  0001 C CNN "Manufacturer_Name"
-F 6 "10%" H 1890 3525 50  0001 C CNN "Tolerance"
+F 4 "CC0603MRX7R8BB104" H 1890 3525 50  0001 C CNN "Manf#"
+F 5 "Yageo" H 1890 3525 50  0001 C CNN "Manufacturer_Name"
+F 6 "20%" H 1890 3525 50  0001 C CNN "Tolerance"
 F 7 "25" H 1890 3525 50  0001 C CNN "voltage"
 	1    1850 3400
@@
 F 2 "Capacitor_SMD:C_0603_1608Metric" H 8350 5550 50  0001 C CNN
 F 3 "" H 8350 5550 50  0001 C CNN
-F 4 "CL10B104KA8NFNC" H 8390 5675 50  0001 C CNN "Manf#"
-F 5 "Samsung" H 8390 5675 50  0001 C CNN "Manufacturer_Name"
-F 6 "10%" H 8390 5675 50  0001 C CNN "Tolerance"
+F 4 "CC0603MRX7R8BB104" H 8390 5675 50  0001 C CNN "Manf#"
+F 5 "Yageo" H 8390 5675 50  0001 C CNN "Manufacturer_Name"
+F 6 "20%" H 8390 5675 50  0001 C CNN "Tolerance"
 F 7 "25" H 8390 5675 50  0001 C CNN "voltage"
 	1    8350 5550
@@
 F 2 "Capacitor_SMD:C_0603_1608Metric" H 1450 4000 50  0001 C CNN
 F 3 "" H 1450 4000 50  0001 C CNN
-F 4 "CL10B104KA8NFNC" H 1490 4125 50  0001 C CNN "Manf#"
-F 5 "Samsung" H 1490 4125 50  0001 C CNN "Manufacturer_Name"
-F 6 "10%" H 1490 4125 50  0001 C CNN "Tolerance"
+F 4 "CC0603MRX7R8BB104" H 1490 4125 50  0001 C CNN "Manf#"
+F 5 "Yageo" H 1490 4125 50  0001 C CNN "Manufacturer_Name"
+F 6 "20%" H 1490 4125 50  0001 C CNN "Tolerance"
 F 7 "25" H 1490 4125 50  0001 C CNN "voltage"
 	1    1450 4000
@@
 F 2 "Capacitor_SMD:C_0603_1608Metric" H 6100 4950 50  0001 C CNN
 F 3 "" H 6100 4950 50  0001 C CNN
-F 4 "CL10B104KA8NFNC" H 6140 5075 50  0001 C CNN "Manf#"
-F 5 "Samsung" H 6140 5075 50  0001 C CNN "Manufacturer_Name"
-F 6 "10%" H 6140 5075 50  0001 C CNN "Tolerance"
+F 4 "CC0603MRX7R8BB104" H 6140 5075 50  0001 C CNN "Manf#"
+F 5 "Yageo" H 6140 5075 50  0001 C CNN "Manufacturer_Name"
+F 6 "20%" H 6140 5075 50  0001 C CNN "Tolerance"
 F 7 "25" H 6140 5075 50  0001 C CNN "voltage"
 	1    6100 4950
