File: junk/adc_gp_backup.sch (KiCad schematic (older format))
At the start: 85 parts, among them IC3 ADS8686SIPZAR

Commit message: changed 0.1uF cap to Samsung
Parts:
- C100, C22, C93, C94, C95, C96, C97, C99: Manf# CL10B104KA8NFNC -> CC0603MRX7R8BB104; Manufacturer_Name Samsung -> Yageo; Tolerance 10% -> 20%
Changed lines of the file:
@@
 F 2 "Capacitor_SMD:C_0603_1608Metric" H 7650 900 50  0001 C CNN
 F 3 "" H 7650 900 50  0001 C CNN
-F 4 "CL10B104KA8NFNC" H 7650 900 50  0001 C CNN "Manf#"
-F 5 "Samsung" H 7700 1100 50  0001 C CNN "Manufacturer_Name"
-F 6 "10%" H 7700 1100 50  0001 C CNN "Tolerance"
+F 4 "CC0603MRX7R8BB104" H 7650 900 50  0001 C CNN "Manf#"
+F 5 "Yageo" H 7700 1100 50  0001 C CNN "Manufacturer_Name"
+F 6 "20%" H 7700 1100 50  0001 C CNN "Tolerance"
 F 7 "25" H 7700 1100 50  0001 C CNN "voltage"
 	1    7650 900
@@
 F 2 "Capacitor_SMD:C_0603_1608Metric" H 8050 900 50  0001 C CNN
 F 3 "" H 8050 900 50  0001 C CNN
-F 4 "CL10B104KA8NFNC" H 8050 900 50  0001 C CNN "Manf#"
-F 5 "Samsung" H 8100 1100 50  0001 C CNN "Manufacturer_Name"
-F 6 "10%" H 8100 1100 50  0001 C CNN "Tolerance"
+F 4 "CC0603MRX7R8BB104" H 8050 900 50  0001 C CNN "Manf#"
+F 5 "Yageo" H 8100 1100 50  0001 C CNN "Manufacturer_Name"
+F 6 "20%" H 8100 1100 50  0001 C CNN "Tolerance"
 F 7 "25" H 8100 1100 50  0001 C CNN "voltage"
 	1    8050 900
@@
 F 2 "Capacitor_SMD:C_0603_1608Metric" H 8450 900 50  0001 C CNN
 F 3 "" H 8450 900 50  0001 C CNN
-F 4 "CL10B104KA8NFNC" H 8450 900 50  0001 C CNN "Manf#"
-F 5 "Samsung" H 8500 1100 50  0001 C CNN "Manufacturer_Name"
-F 6 "10%" H 8500 1100 50  0001 C CNN "Tolerance"
+F 4 "CC0603MRX7R8BB104" H 8450 900 50  0001 C CNN "Manf#"
+F 5 "Yageo" H 8500 1100 50  0001 C CNN "Manufacturer_Name"
+F 6 "20%" H 8500 1100 50  0001 C CNN "Tolerance"
 F 7 "25" H 8500 1100 50  0001 C CNN "voltage"
 	1    8450 900
@@
 F 2 "Capacitor_SMD:C_0603_1608Metric" H 8850 900 50  0001 C CNN
 F 3 "" H 8850 900 50  0001 C CNN
-F 4 "CL10B104KA8NFNC" H 8850 900 50  0001 C CNN "Manf#"
-F 5 "Samsung" H 8900 1100 50  0001 C CNN "Manufacturer_Name"
-F 6 "10%" H 8900 1100 50  0001 C CNN "Tolerance"
+F 4 "CC0603MRX7R8BB104" H 8850 900 50  0001 C CNN "Manf#"
+F 5 "Yageo" H 8900 1100 50  0001 C CNN "Manufacturer_Name"
+F 6 "20%" H 8900 1100 50  0001 C CNN "Tolerance"
 F 7 "25" H 8900 1100 50  0001 C CNN "voltage"
 	1    8850 900
@@
 F 2 "Capacitor_SMD:C_0603_1608Metric" H 9850 950 50  0001 C CNN
 F 3 "" H 9850 950 50  0001 C CNN
-F 4 "CL10B104KA8NFNC" H 9850 950 50  0001 C CNN "Manf#"
-F 5 "Samsung" H 9900 1150 50  0001 C CNN "Manufacturer_Name"
-F 6 "10%" H 9900 1150 50  0001 C CNN "Tolerance"
+F 4 "CC0603MRX7R8BB104" H 9850 950 50  0001 C CNN "Manf#"
+F 5 "Yageo" H 9900 1150 50  0001 C CNN "Manufacturer_Name"
+F 6 "20%" H 9900 1150 50  0001 C CNN "Tolerance"
 F 7 "25" H 9900 1150 50  0001 C CNN "voltage"
 	1    9850 950
@@
 F 2 "Capacitor_SMD:C_0603_1608Metric" H 7900 7000 50  0001 C CNN
 F 3 "" H 7900 7000 50  0001 C CNN
-F 4 "CL10B104KA8NFNC" H 7900 7000 50  0001 C CNN "Manf#"
-F 5 "Samsung" H 8000 7050 50  0001 C CNN "Manufacturer_Name"
-F 6 "10%" H 8000 7050 50  0001 C CNN "Tolerance"
+F 4 "CC0603MRX7R8BB104" H 7900 7000 50  0001 C CNN "Manf#"
+F 5 "Yageo" H 8000 7050 50  0001 C CNN "Manufacturer_Name"
+F 6 "20%" H 8000 7050 50  0001 C CNN "Tolerance"
 F 7 "25" H 8000 7050 50  0001 C CNN "voltage"
 	1    7900 7000
@@
 F 2 "Capacitor_SMD:C_0603_1608Metric" H 10200 4450 50  0001 C CNN
 F 3 "" H 10200 4450 50  0001 C CNN
-F 4 "CL10B104KA8NFNC" H 10200 4450 50  0001 C CNN "Manf#"
-F 5 "Samsung" H 9950 4600 50  0001 C CNN "Manufacturer_Name"
-F 6 "10%" H 9950 4600 50  0001 C CNN "Tolerance"
+F 4 "CC0603MRX7R8BB104" H 10200 4450 50  0001 C CNN "Manf#"
+F 5 "Yageo" H 9950 4600 50  0001 C CNN "Manufacturer_Name"
+F 6 "20%" H 9950 4600 50  0001 C CNN "Tolerance"
 F 7 "25" H 9950 4600 50  0001 C CNN "voltage"
 	1    10200 4450
@@
 F 2 "Capacitor_SMD:C_0603_1608Metric" H 7850 1800 50  0001 C CNN
 F 3 "" H 7850 1800 50  0001 C CNN
-F 4 "CL10B104KA8NFNC" H 7850 1800 50  0001 C CNN "Manf#"
-F 5 "Samsung" H 7900 1950 50  0001 C CNN "Manufacturer_Name"
-F 6 "10%" H 7900 1950 50  0001 C CNN "Tolerance"
+F 4 "CC0603MRX7R8BB104" H 7850 1800 50  0001 C CNN "Manf#"
+F 5 "Yageo" H 7900 1950 50  0001 C CNN "Manufacturer_Name"
+F 6 "20%" H 7900 1950 50  0001 C CNN "Tolerance"
 F 7 "25" H 7900 1950 50  0001 C CNN "voltage"
 	1    7850 1800
