File: junk/dac_backup.sch (KiCad schematic (older format))
At the start: 32 parts, among them IC1 OPA1662, U24 AD5453, U27 OPA2156xD, U35 TMUX6111PWR, U37 OPA2156xD, U8 OPA2156xD

Commit message: changed 0.1uF cap to Samsung
Parts:
- C54, C55, C57, C59, C60: Manf# CL10B104KA8NFNC -> CC0603MRX7R8BB104; Manufacturer_Name Samsung -> Yageo; Tolerance 10% -> 20%
Changed lines of the file:
@@
 F 2 "Capacitor_SMD:C_0603_1608Metric" H 4500 1650 50  0001 C CNN
 F 3 "" H 4500 1650 50  0001 C CNN
-F 4 "CL10B104KA8NFNC" H 4540 1775 50  0001 C CNN "Manf#"
-F 5 "Samsung" H 4540 1775 50  0001 C CNN "Manufacturer_Name"
-F 6 "10%" H 4540 1775 50  0001 C CNN "Tolerance"
+F 4 "CC0603MRX7R8BB104" H 4540 1775 50  0001 C CNN "Manf#"
+F 5 "Yageo" H 4540 1775 50  0001 C CNN "Manufacturer_Name"
+F 6 "20%" H 4540 1775 50  0001 C CNN "Tolerance"
 F 7 "25" H 4540 1775 50  0001 C CNN "voltage"
 	1    4500 1650
@@
 F 2 "Capacitor_SMD:C_0603_1608Metric" H 9000 3100 50  0001 C CNN
 F 3 "" H 9000 3100 50  0001 C CNN
-F 4 "CL10B104KA8NFNC" H 9040 3225 50  0001 C CNN "Manf#"
-F 5 "Samsung" H 9040 3225 50  0001 C CNN "Manufacturer_Name"
-F 6 "10%" H 9040 3225 50  0001 C CNN "Tolerance"
+F 4 "CC0603MRX7R8BB104" H 9040 3225 50  0001 C CNN "Manf#"
+F 5 "Yageo" H 9040 3225 50  0001 C CNN "Manufacturer_Name"
+F 6 "20%" H 9040 3225 50  0001 C CNN "Tolerance"
 F 7 "25" H 9040 3225 50  0001 C CNN "voltage"
 	1    9000 3100
@@
 F 2 "Capacitor_SMD:C_0603_1608Metric" H 7850 3150 50  0001 C CNN
 F 3 "" H 7850 3150 50  0001 C CNN
-F 4 "CL10B104KA8NFNC" H 7890 3275 50  0001 C CNN "Manf#"
-F 5 "Samsung" H 7890 3275 50  0001 C CNN "Manufacturer_Name"
-F 6 "10%" H 7890 3275 50  0001 C CNN "Tolerance"
+F 4 "CC0603MRX7R8BB104" H 7890 3275 50  0001 C CNN "Manf#"
+F 5 "Yageo" H 7890 3275 50  0001 C CNN "Manufacturer_Name"
+F 6 "20%" H 7890 3275 50  0001 C CNN "Tolerance"
 F 7 "25" H 7890 3275 50  0001 C CNN "voltage"
 	1    7850 3150
@@
 F 2 "Capacitor_SMD:C_0603_1608Metric" H 2500 2850 50  0001 C CNN
 F 3 "" H 2500 2850 50  0001 C CNN
-F 4 "CL10B104KA8NFNC" H 2540 2975 50  0001 C CNN "Manf#"
-F 5 "Samsung" H 2540 2975 50  0001 C CNN "Manufacturer_Name"
-F 6 "10%" H 2540 2975 50  0001 C CNN "Tolerance"
+F 4 "CC0603MRX7R8BB104" H 2540 2975 50  0001 C CNN "Manf#"
+F 5 "Yageo" H 2540 2975 50  0001 C CNN "Manufacturer_Name"
+F 6 "20%" H 2540 2975 50  0001 C CNN "Tolerance"
 F 7 "25" H 2540 2975 50  0001 C CNN "voltage"
 	1    2500 2850
@@
 F 2 "Capacitor_SMD:C_0603_1608Metric" H 2500 1850 50  0001 C CNN
 F 3 "" H 2500 1850 50  0001 C CNN
-F 4 "CL10B104KA8NFNC" H 2540 1975 50  0001 C CNN "Manf#"
-F 5 "Samsung" H 2540 1975 50  0001 C CNN "Manufacturer_Name"
-F 6 "10%" H 2540 1975 50  0001 C CNN "Tolerance"
+F 4 "CC0603MRX7R8BB104" H 2540 1975 50  0001 C CNN "Manf#"
+F 5 "Yageo" H 2540 1975 50  0001 C CNN "Manufacturer_Name"
+F 6 "20%" H 2540 1975 50  0001 C CNN "Tolerance"
 F 7 "25" H 2540 1975 50  0001 C CNN "voltage"
 	1    2500 1850
