File: junk/power_backup.sch (KiCad schematic (older format))
At the start: 57 parts, among them J11 Conn_02x05_Odd_Even, J2 PJ-002B, J4 Screw_Terminal_01x12, U11 LT3471, U12 LP38693MP-1.8, U13 LP38693MP-2.5, U14 LP38693MP-5.0, U17 LM2937xMP, U19 MAX6070BAUT21+T, U21 MC79M15_TO252, U5 LP38693MP-3.3

Commit message: changed 0.1uF cap to Samsung
Parts:
- C40, C41, C46, C48, C8: Manf# CL10B104KA8NFNC -> CC0603MRX7R8BB104; Manufacturer_Name Samsung -> Yageo; Tolerance 10% -> 20%
Changed lines of the file:
@@
 F 2 "Capacitor_SMD:C_0603_1608Metric" H 6050 4450 50  0001 C CNN
 F 3 "" H 6050 4450 50  0001 C CNN
-F 4 "CL10B104KA8NFNC" H 6090 4575 50  0001 C CNN "Manf#"
-F 5 "Samsung" H 6090 4575 50  0001 C CNN "Manufacturer_Name"
-F 6 "10%" H 6090 4575 50  0001 C CNN "Tolerance"
+F 4 "CC0603MRX7R8BB104" H 6090 4575 50  0001 C CNN "Manf#"
+F 5 "Yageo" H 6090 4575 50  0001 C CNN "Manufacturer_Name"
+F 6 "20%" H 6090 4575 50  0001 C CNN "Tolerance"
 F 7 "25" H 6090 4575 50  0001 C CNN "voltage"
 	1    6050 4450
@@
 F 2 "Capacitor_SMD:C_0603_1608Metric" H 7250 4400 50  0001 C CNN
 F 3 "" H 7250 4400 50  0001 C CNN
-F 4 "CL10B104KA8NFNC" H 7290 4525 50  0001 C CNN "Manf#"
-F 5 "Samsung" H 7290 4525 50  0001 C CNN "Manufacturer_Name"
-F 6 "10%" H 7290 4525 50  0001 C CNN "Tolerance"
+F 4 "CC0603MRX7R8BB104" H 7290 4525 50  0001 C CNN "Manf#"
+F 5 "Yageo" H 7290 4525 50  0001 C CNN "Manufacturer_Name"
+F 6 "20%" H 7290 4525 50  0001 C CNN "Tolerance"
 F 7 "25" H 7290 4525 50  0001 C CNN "voltage"
 	1    7250 4400
@@
 F 2 "Capacitor_SMD:C_0603_1608Metric" H 8950 5450 50  0001 C CNN
 F 3 "" H 8950 5450 50  0001 C CNN
-F 4 "CL10B104KA8NFNC" H 8990 5575 50  0001 C CNN "Manf#"
-F 5 "Samsung" H 8990 5575 50  0001 C CNN "Manufacturer_Name"
-F 6 "10%" H 8990 5575 50  0001 C CNN "Tolerance"
+F 4 "CC0603MRX7R8BB104" H 8990 5575 50  0001 C CNN "Manf#"
+F 5 "Yageo" H 8990 5575 50  0001 C CNN "Manufacturer_Name"
+F 6 "20%" H 8990 5575 50  0001 C CNN "Tolerance"
 F 7 "25" H 8990 5575 50  0001 C CNN "voltage"
 	1    8950 5450
@@
 F 2 "Capacitor_SMD:C_0603_1608Metric" H 6850 5750 50  0001 C CNN
 F 3 "" H 6850 5750 50  0001 C CNN
-F 4 "CL10B104KA8NFNC" H 6890 5875 50  0001 C CNN "Manf#"
-F 5 "Samsung" H 6890 5875 50  0001 C CNN "Manufacturer_Name"
-F 6 "10%" H 6890 5875 50  0001 C CNN "Tolerance"
+F 4 "CC0603MRX7R8BB104" H 6890 5875 50  0001 C CNN "Manf#"
+F 5 "Yageo" H 6890 5875 50  0001 C CNN "Manufacturer_Name"
+F 6 "20%" H 6890 5875 50  0001 C CNN "Tolerance"
 F 7 "25" H 6890 5875 50  0001 C CNN "voltage"
 	1    6850 5750
@@
 F 2 "Capacitor_SMD:C_0603_1608Metric" H 2000 5100 50  0001 C CNN
 F 3 "" H 2000 5100 50  0001 C CNN
-F 4 "CL10B104KA8NFNC" H 2040 5225 50  0001 C CNN "Manf#"
-F 5 "Samsung" H 2040 5225 50  0001 C CNN "Manufacturer_Name"
-F 6 "10%" H 2040 5225 50  0001 C CNN "Tolerance"
+F 4 "CC0603MRX7R8BB104" H 2040 5225 50  0001 C CNN "Manf#"
+F 5 "Yageo" H 2040 5225 50  0001 C CNN "Manufacturer_Name"
+F 6 "20%" H 2040 5225 50  0001 C CNN "Tolerance"
 F 7 "25" H 2040 5225 50  0001 C CNN "voltage"
 	1    2000 5100
